File: circuit-boards/dual-converter-motherboard-V1.0/dual-converter-motherboard-V1.0.kicad_sch (KiCad schematic)
At the start: 43 parts, among them J1 2601-1102, J10 Conn_02x03_Odd_Even, J11 Conn_02x03_Odd_Even, J12 Conn_02x03_Odd_Even, J13 Conn_02x03_Odd_Even, J14 Conn_02x03_Odd_Even, J2 2601-1102, J3 S4B-XH-SM4-TB, J4 Conn_02x03_Odd_Even, J5 Conn_02x03_Odd_Even, J6 Conn_02x03_Odd_Even, J7 Conn_02x03_Odd_Even, J8 Conn_02x03_Odd_Even, J9 Conn_02x03_Odd_Even, U1 POWER_MANAGEMENT_MODULE, U2 HIGH-CURRENT_PHASE_MODULE_V1.0, U3 HIGH-VOLTAGE_PHASE_MODULE

Commit message: add connectors for non-power pins, improve schematic readability
Parts:
- removed J11: Conn_02x03_Odd_Even, Connector_PinSocket_2.54mm:PinSocket_2x03_P2.54mm_Vertical, symbol Connector_Generic:Conn_02x03_Odd_Even
- added J11, J15: Conn_01x06_Socket, Connector_PinSocket_2.54mm:PinSocket_1x06_P2.54mm_Vertical, symbol Connector:Conn_01x06_Socket
- added J16: Conn_01x07_Socket, Connector_PinSocket_2.54mm:PinSocket_1x07_P2.54mm_Vertical, symbol Connector:Conn_01x07_Socket
Connections:
- net +3.3V: now also J11.1 (Pin_1), J15.1 (Pin_1), J16.5 (Pin_5)
- net +48V: now also J15.5 (Pin_5), J15.6 (Pin_6)
- net BOOST_PGOOD: now also J15.4 (Pin_4)
- net BUCK_ADJ_PWM: now also J16.3 (Pin_3)
- net BUCK_ENABLE: now also J16.2 (Pin_2)
- net BUCK_POWER_GOOD: now also J16.1 (Pin_1)
- net GND: now also J16.4 (Pin_4)
- net I2C_SCL: now also J15.2 (Pin_2), J16.6 (Pin_6)
- net I2C_SDA: now also J15.3 (Pin_3), J16.7 (Pin_7)
- net PMM_DIAG_EN: now also J11.3 (Pin_3)
- net PMM_ENABLE: now also J11.2 (Pin_2)
- net PMM_FAULT: now also J11.4 (Pin_4)
- net PMM_ISENSE: now also J11.5 (Pin_5)
- net PMM_VSENSE: now also J11.6 (Pin_6)
- no-connect marks 1 -> 0
Other:
- moved on the sheet: C1, C2, E1, H1, H10, H11, H12, H13, H14, H15, H16, H17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
