File: circuit-boards/dual-converter-boost-converter-module-V1.0/dual-converter-boost-converter-module-V1.0.kicad_pcb (KiCad board)
At the start: 4 copper layers, 70 x 34 mm, 39 parts, among them J1 Vout Conn, J2 Conn_01x06, J3 Vout Conn, U1 TPL0401B-10DCKR, U2 LM5156HPWPR, U3 STN3N40K3

Commit message: final drc checks, silkscreen edits, added stitching vias to motherboard and pi filter
Routing:
- net +48V: track 20.7 -> 22.7 mm
